File: Front Panel PCB/power_supplies.kicad_sch (KiCad schematic)
At the start: 48 parts, among them J2 Main Power In, J8 Power To Amp, U10 LM317_TO-220, U11 LM337_TO220, U7 LMR36520FADDAR, U8 LMR36520FADDAR, U9 TLV75533PDBVR

Commit message: Checked ERC, assigned all footprints, time to start PCB design, will start with the equiliser
Parts:
- removed COUT3, COUT7: 10u, symbol Device:C_Polarized
- C11, C12, C17, C21, C22, C23, CVCC1, CVCC2: footprint (none) -> GJ821BR71H105KA12L:CAPC2012X135N
- C18, C19, C24, C25, C26, C27, CHF1, CHF2: footprint (none) -> Capacitor_THT:C_Rect_L7.2mm_W2.5mm_P5.00mm
- C20: footprint (none) -> GCM32EC71H106KA03L:CAP_GCM32_MUR
- CIN1, CIN2, CIN3, CIN4: footprint (none) -> GCJ31CC71H475KA01L:CAPC3216X190N
- COUT1, COUT2: value 10u -> 22u; footprint (none) -> GCM32EC71H106KA03L:CAP_GCM32_MUR
- COUT5, COUT6: footprint (none) -> GRM32ER71E226KE15L:G-32_MUR
- J2, J8: footprint (none) -> 1829167:PHOENIX_1829167
- L1: value 33u -> 10u; footprint (none) -> SRP_1038A:IND_SRP1038A_BRN
- L2: footprint (none) -> SRP_1038A:IND_SRP1038A_BRN
- R13, R14, R15, R16, RFBT1, RFBT2: footprint (none) -> Resistor_THT:R_Axial_DIN0207_L6.3mm_D2.5mm_P10.16mm_Horizontal
- RFBB1: footprint (none) -> Resistor_SMD:R_0805_2012Metric
- RFBB2: value 9.09k -> 24.9k; footprint (none) -> Resistor_THT:R_Axial_DIN0207_L6.3mm_D2.5mm_P10.16mm_Horizontal
- U10, U11: footprint Package_TO_SOT_THT:TO-220-3_Vertical -> Package_TO_SOT_THT:TO-220-3_Horizontal_TabDown
Connections:
- net +12V renamed FAN POWER
Other:
- note added: "FAN POWER[5V]"
- note removed: "12V Regulator"
- moved on the sheet: COUT1, COUT2
