File: Front Panel PCB/FrontPanelDesign.kicad_pcb (KiCad board)
At the start: 2 copper layers, 197 parts, among them J1 Conn_01x03_Pin, J10 PA_IN, J11 EQ_OUT, J12 Speakers, J2 Main Power In, J3 LCD I2C, J4 Fan Tach and PWM, J5 Fan Power and GND, J6 VP and VN, J7 DEBUG, J8 Power To Amp, J9 Power In, Q1 BC546, Q10 TIP36, Q11 BC546, Q12 BCM846BS-7, Q13 BC546, Q14 BC546, Q15 BD140, Q16 BC546, Q17 BD139, Q18 BD140, Q19 TIP36, Q2 BC546, Q20 TIP35, Q21 2N3904, Q22 2N7002, Q3 BCM846BS-7, Q4 BC546, Q5 BD140, Q6 BC546, Q7 BD140, Q8 TIP35, Q9 BD139, SW1 SW_Push, U1 TL081, U10 LM317_TO-220, U11 LM337_TO220, U12 STM32G031K8Tx, U2 TL081, U3 TL081, U4 TL081, U5 TL081, U6 TL081, U7 LMR36520FADDAR, U8 LMR36520FADDAR, U9 TLV75533PDBVR

Commit message: Hierarichal sheets and started PCB design
Parts:
- moved C28 233.8 mm to (-60.1, 24.5)
- moved Q3 211.5 mm to (-55.3, 24.6)
- moved C34 193.5 mm to (-51.6, 4.04)
- moved C35 193.5 mm to (-51.6, 8.09)
- moved C37 193.5 mm to (-51.6, 12.1)
- moved RV1 190.8 mm to (-54.9, 19.6)
- moved Q8 178.6 mm to (-94.7, 23.7)
- moved Q10 178.6 mm to (-77.2, 23.7)
- moved R31 176.4 mm to (-61.1, -0.56)
- moved R46 175.3 mm to (89.7, -4.37)
- moved F1 170.5 mm to (-87.7, 45.4)
- moved F2 170.5 mm to (-87.7, 56.5)
- moved C38 161.2 mm to (-95.1, 54.2)
- moved C30 161.0 mm to (-95.1, 30.6)
- moved C32 161.0 mm to (-95.1, 38.5)
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Connections:
- net /AudioL renamed AudioL
- net /AudioR renamed AudioR
- C59 pad 1: unconnected-(C59-Pad1) -> In+
- F1 pad 2: V+ -> VCC
- F2 pad 2: V- -> VEE
- F3 pad 2: V- -> VEE
- F4 pad 2: V+ -> VCC
- J9 pad 1: V- -> VEE
- J9 pad 3: V+ -> VCC
