File: Front Panel PCB/FrontPanelDesign.kicad_sch (KiCad schematic)
At the start: 45 parts, among them J1 Conn_01x03_Pin, J11 EQ_OUT, U1 TL081, U2 TL081, U3 TL081, U4 TL081, U5 TL081, U6 TL081

Commit message: Checked ERC, assigned all footprints, time to start PCB design, will start with the equiliser
Parts:
- C1, C2: footprint (none) -> GCJ31CC71H475KA01L:CAPC3216X190N
- C10, C13, C14, C15, C16, C56, C57, C58, C59, C6, C60, C61, C62, C7, C8, C9: footprint (none) -> Capacitor_THT:C_Rect_L7.2mm_W2.5mm_P5.00mm
- C3, C4, C5: footprint (none) -> ECE_A1HN2R2U:CAPPRD200W50D500H1100
- J1: footprint (none) -> SJ1_3513:CUI_SJ1-3513
- J11: footprint (none) -> Connector_JST:JST_PH_B3B-PH-K_1x03_P2.00mm_Vertical
- R1, R10, R11, R12, R2, R3, R4, R5, R6, R7, R8, R9: footprint (none) -> Resistor_THT:R_Axial_DIN0207_L6.3mm_D2.5mm_P10.16mm_Horizontal
- RV5, RV6, RV7, RV8: footprint (none) -> PTD902:Bourns_PTD902_Dual_Horizontal
- U1, U2, U3, U4, U5, U6: footprint (none) -> Package_DIP:DIP-8_W7.62mm_LongPads
Connections:
- net In+: now also C59.1

Commit message: Hierarichal sheets and started PCB design
Parts:
- removed C1, C2: 4.7u, GCJ31CC71H475KA01L:CAPC3216X190N, symbol Device:C
- removed C10, C15, C56, C57, C58, C59, C60, C61, C62, C7, C8: 100n, Capacitor_THT:C_Rect_L7.2mm_W2.5mm_P5.00mm, symbol Device:C
- removed C13, C14, C16, C6: 22n, Capacitor_THT:C_Rect_L7.2mm_W2.5mm_P5.00mm, symbol Device:C
- removed C3, C4, C5: 2.2u, ECE_A1HN2R2U:CAPPRD200W50D500H1100, symbol Device:C
- removed C9: 1.5n, Capacitor_THT:C_Rect_L7.2mm_W2.5mm_P5.00mm, symbol Device:C
- removed J1: Conn_01x03_Pin, SJ1_3513:CUI_SJ1-3513, symbol Connector:Conn_01x03_Pin
- removed J11: EQ_OUT, Connector_JST:JST_PH_B3B-PH-K_1x03_P2.00mm_Vertical, symbol Connector:Conn_01x02_Pin
- removed R1, R11, R12, R2: 10k, Resistor_THT:R_Axial_DIN0207_L6.3mm_D2.5mm_P10.16mm_Horizontal, symbol Device:R
- removed R10, R3, R5, R8: 470, Resistor_THT:R_Axial_DIN0207_L6.3mm_D2.5mm_P10.16mm_Horizontal, symbol Device:R
- removed R4: 3.3k, Resistor_THT:R_Axial_DIN0207_L6.3mm_D2.5mm_P10.16mm_Horizontal, symbol Device:R
- removed R6, R7, R9: 100k, Resistor_THT:R_Axial_DIN0207_L6.3mm_D2.5mm_P10.16mm_Horizontal, symbol Device:R
- removed RV5, RV6, RV7, RV8: 10k, PTD902:Bourns_PTD902_Dual_Horizontal, symbol Device:R_Potentiometer_Dual
- removed U1, U2, U3, U4, U5, U6: TL081, Package_DIP:DIP-8_W7.62mm_LongPads, symbol Amplifier_Operational:TL081
Connections:
- no-connect marks 13 -> 0
