File: Front Panel PCB/power_amplifier.kicad_sch (KiCad schematic)
At the start: 81 parts, among them J10 PA_IN, J12 Speakers, J9 Power In, Q1 BC546, Q10 TIP36, Q11 BC546, Q12 BCM846BS-7, Q13 BC546, Q14 BC546, Q15 BD140, Q16 BC546, Q17 BD139, Q18 BD140, Q19 TIP36, Q2 BC546, Q20 TIP35, Q3 BCM846BS-7, Q4 BC546, Q5 BD140, Q6 BC546, Q7 BD140, Q8 TIP35, Q9 BD139

Commit message: Checked ERC, assigned all footprints, time to start PCB design, will start with the equiliser
Parts:
- C28, C39: footprint (none) -> GCJ31CC71H475KA01L:CAPC3216X190N
- C29, C31, C40, C42: footprint (none) -> C0805C101J5GACTU:CAPC2012X88N
- C30, C32, C36, C38, C41, C43, C48, C49: footprint (none) -> Capacitor_THT:CP_Radial_D6.3mm_P2.50mm
- C33, C44: footprint (none) -> C0805C301J5GACTU:CAPC2012X88N
- C34, C35, C37, C45, C46, C47: footprint (none) -> Capacitor_THT:C_Rect_L7.2mm_W2.5mm_P5.00mm
- F1, F2, F3, F4: footprint (none) -> Fuse:Fuseholder_Cylinder-5x20mm_Schurter_0031_8201_Horizontal_Open
- J10: footprint (none) -> Connector_JST:JST_PH_B3B-PH-K_1x03_P2.00mm_Vertical
- J12: footprint (none) -> PHOENIX_1757242:PHOENIX_1757242
- J9: footprint (none) -> 1829167:PHOENIX_1829167
- Q10, Q19, Q20, Q8: footprint Package_TO_SOT_THT:TO-220-3_Vertical -> Package_TO_SOT_THT:TO-247-3_Horizontal_TabDown
- Q12, Q3: footprint (none) -> Package_TO_SOT_SMD:SOT-363_SC-70-6
- R17, R18, R19, R20, R21, R22, R23, R24, R25, R26, R27, R30, R32, R33, R34, R35, R36, R37, R38, R39, R40, R41, R42, R43: footprint (none) -> Resistor_THT:R_Axial_DIN0207_L6.3mm_D2.5mm_P10.16mm_Horizontal
- R28, R29, R44, R45: footprint (none) -> Resistor_THT:R_Box_L26.0mm_W5.0mm_P20.00mm
- R31, R46: footprint (none) -> Resistor_THT:R_Axial_DIN0411_L9.9mm_D3.6mm_P15.24mm_Horizontal
- RV1, RV2: footprint (none) -> Potentiometer_THT:Potentiometer_Bourns_3296W_Vertical
Connections:
- net V+ is gone; now on net VCC: F1.2, F4.2, J9.3 (Pin_3)
- net V- renamed VEE

Commit message: Hierarichal sheets and started PCB design
Parts:
- removed C28, C39: 4.7u, GCJ31CC71H475KA01L:CAPC3216X190N, symbol Device:C_Polarized
- removed C29, C31, C40, C42: 100p, C0805C101J5GACTU:CAPC2012X88N, symbol Device:C
- removed C30, C32, C36, C38, C41, C43, C48, C49: 100u, Capacitor_THT:CP_Radial_D6.3mm_P2.50mm, symbol Device:C_Polarized
- removed C33, C44: 300p, C0805C301J5GACTU:CAPC2012X88N, symbol Device:C
- removed C34, C35, C37, C45, C46, C47: 100n, Capacitor_THT:C_Rect_L7.2mm_W2.5mm_P5.00mm, symbol Device:C
- removed F1, F2, F3, F4: T4A, Fuse:Fuseholder_Cylinder-5x20mm_Schurter_0031_8201_Horizontal_Open, symbol Device:Fuse
- removed J10: PA_IN, Connector_JST:JST_PH_B3B-PH-K_1x03_P2.00mm_Vertical, symbol Connector:Conn_01x02_Pin
- removed J12: Speakers, PHOENIX_1757242:PHOENIX_1757242, symbol Connector:Conn_01x02_Pin
- removed J9: Power In, 1829167:PHOENIX_1829167, symbol Connector:Conn_01x03_Pin
- removed Q1, Q11, Q13, Q14, Q16, Q2, Q4, Q6: BC546, Package_TO_SOT_THT:TO-92_Inline, symbol Transistor_BJT:BC546
- removed Q10, Q19: TIP36, Package_TO_SOT_THT:TO-247-3_Horizontal_TabDown, symbol Transistor_BJT:TIP42
- removed Q12, Q3: BCM846BS-7, Package_TO_SOT_SMD:SOT-363_SC-70-6, symbol Transistor_BJT:Q_Dual_NPN_C2C1E1E2
- removed Q15, Q18, Q5, Q7: BD140, Package_TO_SOT_THT:TO-126-3_Vertical, symbol Transistor_BJT:BD140
- removed Q17, Q9: BD139, Package_TO_SOT_THT:TO-126-3_Vertical, symbol Transistor_BJT:BD139
- removed Q20, Q8: TIP35, Package_TO_SOT_THT:TO-247-3_Horizontal_TabDown, symbol Transistor_BJT:TIP41
- removed R17, R19, R22, R32, R34, R39: 1k, Resistor_THT:R_Axial_DIN0207_L6.3mm_D2.5mm_P10.16mm_Horizontal, symbol Device:R
- removed R18, R23, R33, R38: 22k, Resistor_THT:R_Axial_DIN0207_L6.3mm_D2.5mm_P10.16mm_Horizontal, symbol Device:R
- removed R20, R35: 27k, Resistor_THT:R_Axial_DIN0207_L6.3mm_D2.5mm_P10.16mm_Horizontal, symbol Device:R
- removed R21, R37: 1.8k, Resistor_THT:R_Axial_DIN0207_L6.3mm_D2.5mm_P10.16mm_Horizontal, symbol Device:R
- removed R24, R36: 560, Resistor_THT:R_Axial_DIN0207_L6.3mm_D2.5mm_P10.16mm_Horizontal, symbol Device:R
- removed R25, R26, R40, R41: 3.3k, Resistor_THT:R_Axial_DIN0207_L6.3mm_D2.5mm_P10.16mm_Horizontal, symbol Device:R
- removed R27, R30, R42, R43: 270, Resistor_THT:R_Axial_DIN0207_L6.3mm_D2.5mm_P10.16mm_Horizontal, symbol Device:R
- removed R28, R29, R44, R45: .33, Resistor_THT:R_Box_L26.0mm_W5.0mm_P20.00mm, symbol Device:R
- removed R31, R46: 10, Resistor_THT:R_Axial_DIN0411_L9.9mm_D3.6mm_P15.24mm_Horizontal, symbol Device:R
- removed RV1, RV2: 1k, Potentiometer_THT:Potentiometer_Bourns_3296W_Vertical, symbol Device:R_Potentiometer
Other:
- note removed: "A"
- note removed: "B"
