File: Amplifier KiCAD/STM32Setup.kicad_sch (KiCad schematic)
At the start: 25 parts, among them J3 LCD I2C, J4 Fan Tach and PWM, J5 Fan Power and GND, J6 VP and VN, J7 DEBUG, Q21 2N3904, Q22 2N7002, SW1 SW_Push, U12 STM32G031K8Tx

Commit message: Component Placement Finalised, Starting Traces
Parts:
- J5: footprint Connector_Molex:Molex_Micro-Fit_3.0_43045-0812_2x04_P3.00mm_Vertical -> KiCADModels:Molex_Micro-Fit_3.0_43045-0812_2x04_P3.00mm_Vertical
Changed lines of the file:
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@@
 			)
 		)
-		(property "Footprint" "Connector_Molex:Molex_Micro-Fit_3.0_43045-0812_2x04_P3.00mm_Vertical"
+		(property "Footprint" "KiCADModels:Molex_Micro-Fit_3.0_43045-0812_2x04_P3.00mm_Vertical"
 			(at 59.69 152.4 0)
 			(hide yes)
